File: Hardware/DisPhaze.sch (KiCad schematic (older format))
At the start: 78 parts, among them J1 SWD_Header, J2 PItch_In, J3 PD1_Amt_In, J4 PD2_Amt_In, J5 VCA_In, J6 DAC1_Out, J7 DAC2_Out, J8 Eurorack_16_pin_power, SW1 DAC1_RingMod_Switch, SW2 DAC2_Mix_Switch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

Commit message: Added calibration functionality; updated library and startup code
Other:
- note added: "To Do:\nAdd Reset button\nGround Boot0\nCapacitors to VDDA input\nUART/USB IO?"
Changed lines of the file:
@@
 	-1   0    0    1
 $EndComp
+Text Notes 7300 8900 0    50   ~ 0
+To Do:\nAdd Reset button\nGround Boot0\nCapacitors to VDDA input\nUART/USB IO?
 $EndSCHEMATC
