File: Hardware_v3/DisPhaze_Panel.kicad_pcb (KiCad board)
At the start: 2 copper layers, 60.8 x 128.5 mm, 20 parts

Commit message: Updated panel to incorporate v3 redesign
Parts:
- added REF**: USB_Model, Fiducial:Fiducial_0.5mm_Mask1.5mm, F.Cu at (130.0, 136.8)
- added RESET: Subminiature_Switch, Custom_Footprints:Small_Pushbutton_Hole_3.5mm, B.Cu at (130.0, 78.0)
- added Ref**: LED_Hole_3mm, Custom_Footprints:LED_Hole_3mm, B.Cu at (130.0, 62.6)
- moved Ref** 0.06 mm to (105.8, 135.5)
- moved Ref** 0.05 mm to (115.2, 135.5)
Other:
- outline, holes or cut-outs redrawn
- board text added: "DisPhaze Panel v4"
- board text removed: "DisPhaze Panel v3"
Changed lines of the file:
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@@
   )
   (setup
+    (stackup
+      (layer "F.SilkS" (type "Top Silk Screen") (color "White"))
+      (layer "F.Paste" (type "Top Solder Paste"))
+      (layer "F.Mask" (type "Top Solder Mask") (color "Black") (thickness 0.01))
+      (layer "F.Cu" (type "copper") (thickness 0.035))
+      (layer "dielectric 1" (type "core") (thickness 1.51) (material "FR4") (epsilon_r 4.5) (loss_tangent 0.02))
+      (layer "B.Cu" (type "copper") (thickness 0.035))
+      (layer "B.Mask" (type "Bottom Solder Mask") (color "Black") (thickness 0.01))
+      (layer "B.Paste" (type "Bottom Solder Paste"))
+      (layer "B.SilkS" (type "Bottom Silk Screen") (color "White"))
+      (copper_finish "HAL lead-free")
+      (dielectric_constraints no)
+    )
     (pad_to_mask_clearance 0)
     (solder_mask_min_width 0.25)
@@
     (pad "" np_thru_hole oval locked (at 0 0) (size 5 3.2) (drill oval 5 3.2) (layers *.Cu *.Mask))
   )
+  (footprint "Fiducial:Fiducial_0.5mm_Mask1.5mm" (layer "F.Cu")
+    (at 130 136.8)
+    (descr "Circular Fiducial, 0.5mm bare copper, 1.5mm soldermask opening")
+    (tags "fiducial")
+    (attr smd)
+    (fp_text reference "REF**" (at 0 -1.7145) (layer "F.SilkS")
+      (effects (font (size 1 1) (thickness 0.15)))
+    )
+    (fp_text value "USB_Model" (at 0 1.7145) (layer "F.Fab")
+      (effects (font (size 1 1) (thickness 0.15)))
+    )
+    (fp_text user "${REFERENCE}" (at 0 0) (layer "B.Fab")
+      (effects (font (size 0.2 0.2) (thickness 0.04)) (justify mirror))
+    )
+    (model "${CUSTOM_3D}/USB_TE_1734517-1.step"
+      (offset (xyz 0 0 -3))
+      (scale (xyz 1 1 1))
+      (rotate (xyz 0 180 0))
+    )
+  )
   (footprint "Custom_Footprints:Alpha_9mm_pot_hole" (layer "B.Cu")
     (at 147.5 60.51)
@@
   )
   (footprint "Custom_Footprints:Alpha_9mm_pot_hole" (layer "B.Cu")
-    (at 112.5 109.48)
+    (at 112.5 109.5)
     (descr "Mounting Hole 7mm")
     (tags "mounting hole 7mm")
@@
   )
   (footprint "Custom_Footprints:Sub_Miniature_Switch_MountingHole_5mm" (layer "B.Cu")
-    (at 150 135.56)
+    (at 150 135.54)
     (descr "Mounting Hole 6mm, no annular")
     (tags "mounting hole 6mm no annular")
@@
   )
   (footprint "Custom_Footprints:Sub_Miniature_Switch_MountingHole_5mm" (layer "B.Cu")
-    (at 115.25 135.55)
+    (at 115.2 135.54)
     (descr "Mounting Hole 6mm, no annular")
     (tags "mounting hole 6mm no annular")
@@
   )
   (footprint "Custom_Footprints:Sub_Miniature_Switch_MountingHole_5mm" (layer "B.Cu")
-    (at 105.75 135.57)
+    (at 105.8 135.54)
     (descr "Mounting Hole 6mm, no annular")
     (tags "mounting hole 6mm no annular")
@@
       ) (layer "B.Mask") (width 0.01) (fill solid))
   )
+  (footprint "Custom_Footprints:Small_Pushbutton_Hole_3.5mm" (layer "B.Cu")
+    (at 130 78)
+    (descr "Button Hole 3.5mm")
+    (attr through_hole)
+    (fp_text reference "RESET" (at 0 5.4) (layer "B.SilkS") hide
+      (effects (font (size 1 1) (thickness 0.15)) (justify mirror))
+    )
+    (fp_text value "Subminiature_Switch" (at 0 -5.1) (layer "B.Fab") hide
+      (effects (font (size 1 1) (thickness 0.15)) (justify mirror))
+    )
+    (fp_circle (center 0 0) (end 1.5 0) (layer "Cmts.User") (width 0.15) (fill none))
+    (fp_circle (center 0 0) (end 1.6 0) (layer "B.CrtYd") (width 0.05) (fill none))
+    (pad "" np_thru_hole circle locked (at 0 0) (size 3.5 3.5) (drill 3.5) (layers *.Cu *.Mask))
+    (model "${KISYS3DMOD}/Button_Switch_THT.3dshapes/SW_PUSH_6mm_H13mm.wrl"
+      (offset (xyz -3.15 2.25 -11.5))
+      (scale (xyz 1 1 1))
+      (rotate (xyz 0 0 0))
+    )
+  )
+  (footprint "Custom_Footprints:LED_Hole_3mm" (layer "B.Cu")
+    (at 130 62.6 180)
+    (descr "Mounting Hole 6mm, no annular")
+    (tags "mounting hole 6mm no annular")
+    (attr through_hole)
+    (fp_text reference "Ref**" (at 0 5.4) (layer "B.SilkS") hide
+      (effects (font (size 1 1) (thickness 0.15)) (justify mirror))
+    )
+    (fp_text value "LED_Hole_3mm" (at 0 -5.1) (layer "B.Fab") hide
+      (effects (font (size 1 1) (thickness 0.15)) (justify mirror))
+    )
+    (fp_circle (center 0 0) (end 1.5 0) (layer "Cmts.User") (width 0.1) (fill none))
+    (fp_circle (center 0 0) (end 1.6 0) (layer "B.CrtYd") (width 0.05) (fill none))
+    (pad "" np_thru_hole circle locked (at 0 0 180) (size 3 3) (drill 3) (layers *.Cu *.Mask))
+    (model "${KISYS3DMOD}/LED_THT.3dshapes/LED_D3.0mm_FlatTop.wrl"
+      (offset (xyz -1.27 0 -8.3))
+      (scale (xyz 1 1 1))
+      (rotate (xyz 0 0 0))
+    )
+  )
   (gr_line (start 112.5 100.25) (end 112.5 102.1) (layer "B.Mask") (width 0.5))
   (gr_poly
@@
   (gr_line (start 130 120.6) (end 134.1 124.9) (layer "B.Mask") (width 0.3))
   (gr_line (start 125.9 124.9) (end 130 120.6) (layer "B.Mask") (width 0.3))
-  (gr_line (start 130.1 53.2) (end 130.1 91.2) (layer "B.Mask") (width 0.3))
-  (gr_line (start 130 129.7) (end 130 143.3) (layer "B.Mask") (width 0.3))
+  (gr_line (start 130 64.9) (end 130 75.7) (layer "B.Mask") (width 0.3))
   (gr_line (start 155 152) (end 145 152) (layer "B.Mask") (width 0.3))
   (gr_line (start 115 152) (end 105 152) (layer "B.Mask") (width 0.3))
   (gr_arc (start 156.080946 106.748093) (mid 156.486223 110.173372) (end 155.575 113.5) (layer "B.Mask") (width 0.4))
+  (gr_line (start 130 80.3) (end 130 91.2) (layer "B.Mask") (width 0.3))
+  (gr_line (start 130 53.2) (end 130 60.3) (layer "B.Mask") (width 0.3))
+  (gr_circle (center 130 62.6) (end 132.3 62.6) (layer "B.Mask") (width 0.2) (fill none))
   (gr_poly
     (pts
@@
       (xy 109.5 147.5)
     ) (layer "B.Mask") (width 0.1) (fill solid))
+  (gr_circle (center 130 78) (end 132.3 78) (layer "B.Mask") (width 0.2) (fill none))
   (gr_line (start 100 160) (end 160 160) (layer "Dwgs.User") (width 0.2))
   (gr_line (start 160 50) (end 160 160) (layer "Dwgs.User") (width 0.2))
@@
   (gr_line (start 99.6 169.3) (end 160.4 169.3) (layer "Edge.Cuts") (width 0.1))
   (gr_line (start 99.6 40.8) (end 160.4 40.8) (layer "Edge.Cuts") (width 0.1))
+  (gr_rect (start 123.8 130.9) (end 136.2 142.7) (layer "Edge.Cuts") (width 0.1) (fill none))
   (gr_line (start 160.4 40.8) (end 160.4 169.3) (layer "Edge.Cuts") (width 0.1))
   (gr_text "CZ Peasy" (at 130.5 43.25) (layer "F.SilkS")
@@
     (effects (font (size 1 1) (thickness 0.15)))
   )
-  (gr_text "DisPhaze Panel v3" (at 130.5 167) (layer "F.SilkS")
+  (gr_text "DisPhaze Panel v4" (at 130.5 167) (layer "F.SilkS")
     (effects (font (size 1.5 1.5) (thickness 0.3)))
   )
@@
   (zone (net 0) (net_name "") (layer "F.Cu") (hatch edge 0.508)
     (connect_pads (clearance 0.508))
-    (min_thickness 0.254)
+    (min_thickness 0.254) (filled_areas_thickness no)
     (fill yes (thermal_gap 0.508) (thermal_bridge_width 0.508))
     (polygon
@@
   (zone (net 0) (net_name "") (layer "B.Cu") (hatch edge 0.508)
     (connect_pads (clearance 0.508))
-    (min_thickness 0.254)
+    (min_thickness 0.254) (filled_areas_thickness no)
     (fill yes (thermal_gap 0.508) (thermal_bridge_width 0.508))
     (polygon

Commit message: Preparation of Gerbers for v3 hardware ordering
Parts:
- added kibuzzard-623877CE: G***, kibuzzard-623877CE, B.Cu at (125.0, 145.5)
- added kibuzzard-623877D8: G***, kibuzzard-623877D8, B.Cu at (135.1, 145.5)
