File: Hardware_v3/DisPhaze_Components.kicad_sch (KiCad schematic)
At the start: 89 parts, among them J1 SWD_Header, J2 USB_B_Micro, J3 PItch_In, J4 PD1_Amt_In, J5 PD2_Amt_In, J6 VCA_In, J7 DAC1_Out, J8 DAC2_Out, J9 Eurorack_16_pin_power, Q1 MMBT3904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

Commit message: Gpio class button handles both pull up/down
Also added pull downs to switch pins
Parts:
- R4: value 91k -> 82k
- R5: value 56k -> 47k
Changed lines of the file:
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@@
 	(wire
 		(pts
-			(xy 260.35 189.23) (xy 266.7 189.23)
+			(xy 260.35 189.23) (xy 264.16 189.23)
 		)
 		(stroke
@@
 	(wire
 		(pts
-			(xy 260.35 167.64) (xy 266.7 167.64)
+			(xy 260.35 167.64) (xy 264.16 167.64)
 		)
 		(stroke
@@
 	(wire
 		(pts
+			(xy 260.35 212.09) (xy 264.16 212.09)
+		)
+		(stroke
+			(width 0)
+			(type default)
+		)
+	)
+	(wire
+		(pts
 			(xy 93.98 250.19) (xy 81.28 250.19)
 		)
@@
 	(wire
 		(pts
-			(xy 260.35 212.09) (xy 266.7 212.09)
-		)
-		(stroke
-			(width 0)
-			(type default)
-		)
-	)
-	(wire
-		(pts
 			(xy 267.335 95.25) (xy 267.335 97.79)
 		)
@@
 	(wire
 		(pts
-			(xy 266.7 165.1) (xy 266.7 167.64)
+			(xy 264.16 166.37) (xy 264.16 167.64)
 		)
 		(stroke
@@
 	(wire
 		(pts
-			(xy 266.7 186.69) (xy 266.7 189.23)
+			(xy 264.16 187.96) (xy 264.16 189.23)
 		)
 		(stroke
@@
 	(wire
 		(pts
-			(xy 266.7 209.55) (xy 266.7 212.09)
+			(xy 264.16 210.82) (xy 264.16 212.09)
 		)
 		(stroke
@@
 			)
 		)
-		(property "Value" "56k"
+		(property "Value" "47k"
 			(at 167.64 31.9786 90)
 			(effects
@@
 			)
 		)
-		(property "Value" "91k"
+		(property "Value" "82k"
 			(at 154.94 23.0886 90)
 			(effects
@@
 	(symbol
 		(lib_id "power:+3.3V")
-		(at 266.7 165.1 0)
+		(at 264.16 166.37 0)
 		(unit 1)
 		(exclude_from_sim no)
@@
 		(dnp no)
 		(property "Reference" "#PWR031"
-			(at 266.7 168.91 0)
+			(at 264.16 170.18 0)
 			(effects
 				(font
@@
 		)
 		(property "Value" "+3V3"
-			(at 267.081 160.7058 0)
+			(at 264.541 161.9758 0)
 			(effects
 				(font
@@
 		)
 		(property "Footprint" ""
-			(at 266.7 165.1 0)
+			(at 264.16 166.37 0)
 			(effects
 				(font
@@
 		)
 		(property "Datasheet" ""
-			(at 266.7 165.1 0)
+			(at 264.16 166.37 0)
 			(effects
 				(font
@@
 		)
 		(property "Description" ""
-			(at 266.7 165.1 0)
+			(at 264.16 166.37 0)
 			(effects
 				(font
@@
 	(symbol
 		(lib_id "power:+3.3V")
-		(at 266.7 209.55 0)
+		(at 264.16 210.82 0)
 		(unit 1)
 		(exclude_from_sim no)
@@
 		(dnp no)
 		(property "Reference" "#PWR035"
-			(at 266.7 213.36 0)
+			(at 264.16 214.63 0)
 			(effects
 				(font
@@
 		)
 		(property "Value" "+3V3"
-			(at 267.081 205.1558 0)
+			(at 264.541 206.4258 0)
 			(effects
 				(font
@@
 		)
 		(property "Footprint" ""
-			(at 266.7 209.55 0)
+			(at 264.16 210.82 0)
 			(effects
 				(font
@@
 		)
 		(property "Datasheet" ""
-			(at 266.7 209.55 0)
+			(at 264.16 210.82 0)
 			(effects
 				(font
@@
 		)
 		(property "Description" ""
-			(at 266.7 209.55 0)
+			(at 264.16 210.82 0)
 			(effects
 				(font
@@
 	(symbol
 		(lib_id "power:+3.3V")
-		(at 266.7 186.69 0)
+		(at 264.16 187.96 0)
 		(unit 1)
 		(exclude_from_sim no)
@@
 		(dnp no)
 		(property "Reference" "#PWR033"
-			(at 266.7 190.5 0)
+			(at 264.16 191.77 0)
 			(effects
 				(font
@@
 		)
 		(property "Value" "+3V3"
-			(at 267.081 182.2958 0)
+			(at 264.541 183.5658 0)
 			(effects
 				(font
@@
 		)
 		(property "Footprint" ""
-			(at 266.7 186.69 0)
+			(at 264.16 187.96 0)
 			(effects
 				(font
@@
 		)
 		(property "Datasheet" ""
-			(at 266.7 186.69 0)
+			(at 264.16 187.96 0)
 			(effects
 				(font
@@
 		)
 		(property "Description" ""
-			(at 266.7 186.69 0)
+			(at 264.16 187.96 0)
 			(effects
 				(font

Commit message: Fixes to LED handling
Other:
- note added: "HP Input filter cutoff .34Hz"
Changed lines of the file:
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@@
+		)
+	)
+	(text "HP Input filter cutoff .34Hz"
+		(exclude_from_sim no)
+		(at 265.684 117.602 0)
+		(effects
+			(font
+				(size 1.27 1.27)
+			)
 		)
 	)
