File: Hardware_v3/DisPhaze_Components.kicad_sch (KiCad schematic)
At the start: 89 parts, among them J1 SWD_Header, J2 USB_B_Micro, J3 PItch_In, J4 PD1_Amt_In, J5 PD2_Amt_In, J6 VCA_In, J7 DAC1_Out, J8 DAC2_Out, J9 Eurorack_16_pin_power, Q1 MMBT3904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

Commit message: More handling for MIDI issues
Parts:
- C16: value 22pF -> 1nF
- C18: value 22pF -> 1nf
- R17, R21: value 68k -> 10k
- R18, R22: value 6.8k -> 2k
Other:
- note added: "HP Input filter cutoff .34Hz Post HP filter levels are -1.3V > +1.3V Gain = x5 (10k/2k) output -6.5V > 6.5V LP Feedback filter cut off: 1 / 2πR_{f}C_{f} = 16KHz"
- note added: "v3 Errata - CV Incorrectly normalled to V/Oct - Change Eurorack connector to 10 pin? - Add UART header - DACs swapped - OUtput amplifier values changed (done)"
- note removed: "HP Input filter cutoff .34Hz LP Feedback filter: 1 / 2πR_{f}C_{f}"
- note removed: "v3 Errata - CV Incorrectly normalled to V/Oct - Change Eurorack connector to 10 pin? - Add UART header - Problems connecting Action button to 3.3V - change to GND"
Changed lines of the file:
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@@
 		)
 	)
-	(text "v3 Errata\n- CV Incorrectly normalled to V/Oct\n- Change Eurorack connector to 10 pin?\n- Add UART header\n- Problems connecting Action button to 3.3V - change to GND"
+	(text "v3 Errata\n- CV Incorrectly normalled to V/Oct\n- Change Eurorack connector to 10 pin?\n- Add UART header\n- DACs swapped\n- OUtput amplifier values changed (done)"
 		(exclude_from_sim no)
-		(at 309.88 257.81 0)
+		(at 304.8 259.08 0)
 		(effects
 			(font
@@
 		)
 	)
-	(text "HP Input filter cutoff .34Hz\nLP Feedback filter: 1 / 2πR_{f}C_{f}"
+	(text "HP Input filter cutoff .34Hz\nPost HP filter levels are -1.3V > +1.3V\nGain = x5 (10k/2k) output -6.5V > 6.5V\nLP Feedback filter cut off: 1 / 2πR_{f}C_{f} = 16KHz"
 		(exclude_from_sim no)
 		(at 265.684 117.602 0)
@@
 			)
 		)
-		(property "Value" "68k"
+		(property "Value" "10k"
 			(at 245.11 79.6036 90)
 			(effects
@@
 			)
 		)
-		(property "Value" "6.8k"
+		(property "Value" "2k"
 			(at 232.41 87.2236 90)
 			(effects
@@
 			)
 		)
-		(property "Value" "68k"
+		(property "Value" "10k"
 			(at 245.11 31.9786 90)
 			(effects
@@
 			)
 		)
-		(property "Value" "6.8k"
+		(property "Value" "2k"
 			(at 232.41 40.2336 90)
 			(effects
@@
 			)
 		)
-		(property "Value" "22pF"
+		(property "Value" "1nf"
 			(at 245.11 69.5706 90)
 			(effects
@@
 			)
 		)
-		(property "Value" "22pF"
+		(property "Value" "1nF"
 			(at 245.11 21.3106 90)
 			(effects
